File: hardware/DAC_HPA_100x80_REVIEW_ONLY.kicad_pcb (KiCad board)
At the start: 4 copper layers, 100 x 80 mm, 537 parts, among them J101 GCT USB4105-GF-A, J201 PCB pads (no component), J202 PCB pads (no component), J701 G-Switch GT-3321667P-01, J702 HRO PJ-332A-6A, J703 1 × 6, K601 TLP3545A, K602 TLP3545A, K603 TLP3545A, K604 TLP3545A, Q207 AO3400A, Q502 AO3400A, Q503 AO3400A, Q504 AO3400A, Q505 AO3400A, Q506 AO3400A, Q507 MMBT3904, Q612 MMBT3904, Q614 MMBT3904, Q616 AO3400A, Q617 AO3400A, Q618 2N7002, Q619 AO3400A, Q620 AO3400A, Q621 2N7002, Q622 AO3400A, Q623 MMBT3904, Q624 MMBT3904, Q625 MMBT3904, Q626 MMBT3904, Q627 MMBT3904, U101 ST USBLC6-2SC6, U102 TI TPS25200DRVR, U103 TI TPD2E2U06DRLR, U201 CH32V307RCT6, U202 AGRV2KQ32, U205 74LVC1G157, U206 74LVC1G11, U208 74LVC3G34, U301 ES9018K2M, U302 3.3 V, 250 mA, U303 1.300 V (R533/R534), U401 OPA1622IDRCR, U402 OPA1622IDRCR, U403 OPA2210IDGKR, U404 OPA2210IDGKR, U501 +3.85 / -3.72 V, U502 3.3 V, 150 mA, U503 TI TPS259621DDAR, U504 3.3 V, 1 A, U505 TI TMUX1101DBVR, U603 TLV1704, U604 OPA2333, U605 TLV3402, U606 TLV1704, U607 74AUP1G17, U608 74LVC1G74, U609 TLV1704, U610 TLV1704, U611 TLV1704, U612 TLV1704, U613 TLV3402, U614 TLV3402, U615 TLV3402, U616 TLV3402, U617 TLV3402, U618 TLV3402, U619 TLV3402, U620 TLV3402, X201 80.000 MHz, X202 49.152 MHz, X203 45.1584 MHz, Y201 8 MHz

Commit message: Manually review 120x100 layout with JLCPCB rules and ESD escapes
Parts:
- removed J703: 1 × 6, Connector_PinHeader_2.54mm:PinHeader_2x03_P2.54mm_Vertical
