File: hardware/06_protection.kicad_sch (KiCad schematic)
At the start: 167 parts, among them K601 TLP3545A, K602 TLP3545A, K603 TLP3545A, K604 TLP3545A, Q612 MMBT3904, Q614 MMBT3904, Q616 AO3400A, Q617 AO3400A, Q618 2N7002, Q619 AO3400A, Q620 AO3400A, Q621 2N7002, Q622 AO3400A, Q623 MMBT3904, Q624 MMBT3904, Q625 MMBT3904, Q626 MMBT3904, U601 TLV1704, U602 TLV1704, U603 TLV1704, U604 OPA2333, U605 TLV3402, U606 TLV1704, U607 74AUP1G17, U608 74LVC1G74, U609 TLV1704, U610 TLV1704

Commit message: Recapture DAC-HPA schematic for design set v1.1
Parts:
- removed C601, C602, C603, C604: 2.2 µF, Capacitor_SMD:C_0603_1608Metric, symbol DAC_HPA:P122
- removed C612, C613, C614, C615: 100 nF, Capacitor_SMD:C_0402_1005Metric, symbol DAC_HPA:P124
- removed R601, R602, R603, R604: 115 kΩ, Resistor_SMD:R_0402_1005Metric, symbol DAC_HPA:P137
- removed R607: 121 kΩ, Resistor_SMD:R_0402_1005Metric, symbol DAC_HPA:P138
- removed R608: 115 kΩ, Resistor_SMD:R_0402_1005Metric, symbol DAC_HPA:P139
- removed R609, R610: 10.0 kΩ, Resistor_SMD:R_0402_1005Metric, symbol DAC_HPA:P140
- removed R649, R650, R651, R652: 100 kΩ, Resistor_SMD:R_0402_1005Metric, symbol DAC_HPA:P147
- removed U601, U602: TLV1704, JLC_Imported:TSSOP-14_L5.0-W4.4-P0.65-LS6.4-BL, symbol DAC_HPA:P165
- added C639, C640, C641, C642: 1 nF, Capacitor_SMD:C_0402_1005Metric, symbol DAC_HPA:P128
- added C643, C644, C645, C646: 3.3 nF, Capacitor_SMD:C_0603_1608Metric, symbol DAC_HPA:P130
- added C647, C648, C649, C650, C651, C652, C653, C654: 100 nF, Capacitor_SMD:C_1206_3216Metric, symbol DAC_HPA:P131
- added C655, C656, C657, C658, C659, C660, C661, C662, C663, C664, C665, C666: 100 nF, Capacitor_SMD:C_0402_1005Metric, symbol DAC_HPA:P124
- added Q627: MMBT3904, JLC_Imported:SOT-23-3_L2.9-W1.6-P1.90-LS2.8-BR, symbol DAC_HPA:P137
- added R926, R927, R928, R929: 330 kΩ, Resistor_SMD:R_0402_1005Metric, symbol DAC_HPA:P147
- added R930, R931, R932, R933, R938, R940: 1.00 MΩ, Resistor_SMD:R_0402_1005Metric, symbol DAC_HPA:P149
- added R934: 360 kΩ, Resistor_SMD:R_0402_1005Metric, symbol DAC_HPA:P163
- added R935, R936, R937: 470 kΩ, Resistor_SMD:R_0402_1005Metric, symbol DAC_HPA:P159
- added R939, R950: 100 kΩ, Resistor_SMD:R_0402_1005Metric, symbol DAC_HPA:P144
- added R941: 88.7 kΩ, Resistor_SMD:R_0402_1005Metric, symbol DAC_HPA:P164
- added R942, R943, R944, R945, R946, R947, R948, R949: 910 kΩ, Resistor_SMD:R_0402_1005Metric, symbol DAC_HPA:P165
- added R951: 10 kΩ, Resistor_SMD:R_0402_1005Metric, symbol DAC_HPA:P166
- added U611, U612: TLV1704, JLC_Imported:TSSOP-14_L5.0-W4.4-P0.65-LS6.4-BL, symbol DAC_HPA:P167
- added U613, U614, U615, U616, U617, U618, U619, U620: TLV3402, JLC_Imported:VSSOP-8_L3.0-W3.0-P0.65-LS5.0-BL, symbol DAC_HPA:P172
- C608, C609, C610, C611, C616: symbol DAC_HPA:P123 -> DAC_HPA:P122
- C617: symbol DAC_HPA:P125 -> DAC_HPA:P123
- C620, C621: symbol DAC_HPA:P126 -> DAC_HPA:P125
- C624: symbol DAC_HPA:P127 -> DAC_HPA:P126
- C625: symbol DAC_HPA:P128 -> DAC_HPA:P127
- C629: symbol DAC_HPA:P129 -> DAC_HPA:P128
- C631, C632, C633, C634: symbol DAC_HPA:P130 -> DAC_HPA:P129
- D609, D610: symbol DAC_HPA:P131 -> DAC_HPA:P132
- K601, K602, K603, K604: symbol DAC_HPA:P132 -> DAC_HPA:P133
- Q612, Q614: symbol DAC_HPA:P133 -> DAC_HPA:P134
- Q616, Q617, Q619, Q620, Q622: symbol DAC_HPA:P134 -> DAC_HPA:P135
- Q618, Q621: symbol DAC_HPA:P135 -> DAC_HPA:P136
- Q623, Q624, Q625, Q626: footprint JLC_Imported:SOT-23-3_L2.9-W1.3-P1.90-LS2.4-BR -> JLC_Imported:SOT-23-3_L2.9-W1.6-P1.90-LS2.8-BR; symbol DAC_HPA:P136 -> DAC_HPA:P137; LCSC C20526 -> C81464; LCSC Part # C20526 -> C81464; MPN JSCJ MMBT3904 (RANGE:100-300) -> onsemi MMBT3904LT1G; Rating/Tolerance 40 V, 200 mA; VCE(sat) ≤ 0.2 V; ICBO ≤ 50 nA; VEB 6 V -> 40 V, 200 mA; VCE(sat) ≤ 0.2 V at 10 mA / 1 mA, ≤ 0.3 V at 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
- R624, R625, R626, R627, R658, R661: symbol DAC_HPA:P141 -> DAC_HPA:P138
- R628, R629, R630, R631, R639, R663: symbol DAC_HPA:P142 -> DAC_HPA:P139
- R632, R633, R634, R635, R640: symbol DAC_HPA:P143 -> DAC_HPA:P140
- R641, R642: symbol DAC_HPA:P144 -> DAC_HPA:P141
- R643, R644: symbol DAC_HPA:P145 -> DAC_HPA:P142
- R645, R692: symbol DAC_HPA:P146 -> DAC_HPA:P143
- R646, R647, R648, R667, R669, R680, R687, R691, R693, R695, R696: symbol DAC_HPA:P147 -> DAC_HPA:P144
- R653, R654, R655, R656, R662, R673, R925: symbol DAC_HPA:P148 -> DAC_HPA:P145
- R657, R659, R670: symbol DAC_HPA:P140 -> DAC_HPA:P146
- R660, R690, R694, R916, R917, R918, R919: symbol DAC_HPA:P149 -> DAC_HPA:P147
- R665: symbol DAC_HPA:P150 -> DAC_HPA:P148
- R666, R668: symbol DAC_HPA:P151 -> DAC_HPA:P149
- R671: symbol DAC_HPA:P152 -> DAC_HPA:P150
- R672: symbol DAC_HPA:P153 -> DAC_HPA:P151
- R674: symbol DAC_HPA:P154 -> DAC_HPA:P152
- R675, R682: symbol DAC_HPA:P155 -> DAC_HPA:P153
- R676, R683: symbol DAC_HPA:P156 -> DAC_HPA:P154
- R677, R684: symbol DAC_HPA:P157 -> DAC_HPA:P155
- R678, R685, R901, R903, R905, R907, R909, R911, R913, R915: symbol DAC_HPA:P158 -> DAC_HPA:P156
- R679, R686: symbol DAC_HPA:P159 -> DAC_HPA:P157
- R681: symbol DAC_HPA:P160 -> DAC_HPA:P158
- R688, R689: symbol DAC_HPA:P161 -> DAC_HPA:P159
- R900, R902, R904, R906, R908, R910, R912, R914: symbol DAC_HPA:P162 -> DAC_HPA:P160
- R920, R921, R922, R923: symbol DAC_HPA:P163 -> DAC_HPA:P161
- R924: symbol DAC_HPA:P164 -> DAC_HPA:P162
- U603, U606, U609, U610: symbol DAC_HPA:P165 -> DAC_HPA:P167
- U604: symbol DAC_HPA:P166 -> DAC_HPA:P168
- U605: symbol DAC_HPA:P167 -> DAC_HPA:P169
- U607: symbol DAC_HPA:P168 -> DAC_HPA:P170
- U608: symbol DAC_HPA:P169 -> DAC_HPA:P171
Connections:
- net 3V3A: now also R934.1, R938.1
- net GND: now also C639.2, C640.2, C641.2, C642.2, C643.2, C644.2, C645.2, C646.2, C647.2, C648.2, C649.2, C650.2, C651.2, C652.2, C653.2, C654.2, C655.2, C656.2, C657.2, C658.2, Q627.2 (E), R935.2, R939.2, R941.2, U613.5 (IN2+), U614.5 (IN2+), U615.5 (IN2+), U616.5 (IN2+), U617.5 (IN2+), U618.5 (IN2+), U619.5 (IN2+), U620.5 (IN2+)
- net LEG_LN: now also R927.1, R931.1
- net LEG_LP: now also R926.1, R930.1
- net LEG_RN: now also R929.1, R933.1
- net LEG_RP: now also R928.1, R932.1
- net N6_OLN_L: now also U611.1 (2OUT), U611.14 (3OUT), U614.7 (OUT2), U615.7 (OUT2)
- net N6_OLN_R: now also U612.1 (2OUT), U612.14 (3OUT), U618.7 (OUT2), U619.7 (OUT2)
- net N6_OLP_L: now also U611.13 (4OUT), U611.2 (1OUT), U613.7 (OUT2), U616.7 (OUT2)
- net N6_OLP_R: now also U612.13 (4OUT), U612.2 (1OUT), U617.7 (OUT2), U620.7 (OUT2)
- net VNEG: now also C656.1, C658.1, C659.2, C660.2, C661.2, C662.2, C663.2, C664.2, C665.2, C666.2, R936.1, R940.1, U611.12 (V-), U612.12 (V-), U613.4 (GND), U614.4 (GND), U615.4 (GND), U616.4 (GND), U617.4 (GND), U618.4 (GND), U619.4 (GND), U620.4 (GND)
- net VPOS: now also C655.1, C657.1, C659.1, C660.1, C661.1, C662.1, C663.1, C664.1, C665.1, C666.1, R942.1, R943.1, R944.1, R945.1, R946.1, R947.1, R948.1, R949.1, U611.3 (V+), U612.3 (V+), U613.8 (VCC), U614.8 (VCC), U615.8 (VCC), U616.8 (VCC), U617.8 (VCC), U618.8 (VCC), U619.8 (VCC), U620.8 (VCC)
- new net N6_LWLN: C644.1, R931.2, U615.3 (IN1+), U616.2 (IN1-)
- new net N6_LWLP: C643.1, R930.2, U613.3 (IN1+), U614.2 (IN1-)
- new net N6_LWRN: C646.1, R933.2, U619.3 (IN1+), U620.2 (IN1-)
- new net N6_LWRP: C645.1, R932.2, U617.3 (IN1+), U618.2 (IN1-)
- new net N6_ORLN: C640.1, R927.2, U611.11 (4IN+), U611.8 (3IN-)
- new net N6_ORLP: C639.1, R926.2, U611.4 (1IN-), U611.7 (2IN+)
- new net N6_ORQC: Q627.3 (C), R951.2
- new net N6_ORRN: C642.1, R929.2, U612.11 (4IN+), U612.8 (3IN-)
- new net N6_ORRP: C641.1, R928.2, U612.4 (1IN-), U612.7 (2IN+)
- new net N6_ORTB: Q627.1 (B), R950.2
- new net N6_ORTEST: R937.2, R950.1
- new net N6_TWLNN: C650.1, R945.2, U616.1 (OUT1), U616.6 (IN2-)
- new net N6_TWLNP: C649.1, R944.2, U615.1 (OUT1), U615.6 (IN2-)
- new net N6_TWLPN: C648.1, R943.2, U614.1 (OUT1), U614.6 (IN2-)
- new net N6_TWLPP: C647.1, R942.2, U613.1 (OUT1), U613.6 (IN2-)
- new net N6_TWRNN: C654.1, R949.2, U620.1 (OUT1), U620.6 (IN2-)
- new net N6_TWRNP: C653.1, R948.2, U619.1 (OUT1), U619.6 (IN2-)
- new net N6_TWRPN: C652.1, R947.2, U618.1 (OUT1), U618.6 (IN2-)
- new net N6_TWRPP: C651.1, R946.2, U617.1 (OUT1), U617.6 (IN2-)
- new net N6_VLLN: R940.2, R941.1, U614.3 (IN1+), U616.3 (IN1+), U618.3 (IN1+), U620.3 (IN1+)
- new net N6_VLLP: R938.2, R939.1, U613.2 (IN1-), U615.2 (IN1-), U617.2 (IN1-), U619.2 (IN1-)
- new net N6_VORN: R936.2, R937.1, U611.10 (4IN-), U611.6 (2IN-), U612.10 (4IN-), U612.6 (2IN-)
- new net N6_VORP: R934.2, R935.1, R951.1, U611.5 (1IN+), U611.9 (3IN+), U612.5 (1IN+), U612.9 (3IN+)
Other:
- moved on the sheet: C608, C609, C610, C611, C616, C617, C618, C619, C620, C621, C622, C623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

Commit message: Capture functional ECO and manual 120x100 review board
Parts:
- added C667: 100 nF, Capacitor_SMD:C_0402_1005Metric, symbol DAC_HPA:P9004
- added R952, R953: 10 kΩ, Resistor_SMD:R_0402_1005Metric, symbol DAC_HPA:P9002
- added R954, R955: 100 kΩ, Resistor_SMD:R_0402_1005Metric, symbol DAC_HPA:P9003
- added U621: SN74AUP2G17DCKR, JLC_Imported:SC-70-6_L2.2-W1.3-P0.65-LS2.1-BL, symbol DAC_HPA:P9001
Connections:
- net 3V3M: now also C667.1, R954.1, R955.1, U621.5 (VCC)
- net GND: now also C667.2, U621.2 (GND)
- net N6_V3AG_A_MCU: now also R952.2, R954.2; no longer R688.2
- net N6_V3AG_B_MCU: now also R953.2, R955.2; no longer R689.2
- new net N6_V3AG_A_BUF_IN: R688.2, U621.1 (1A)
- new net N6_V3AG_A_BUF_OUT: R952.1, U621.6 (1Y)
- new net N6_V3AG_B_BUF_IN: R689.2, U621.3 (2A)
- new net N6_V3AG_B_BUF_OUT: R953.1, U621.4 (2Y)
Other:
- moved on the sheet: R688, R689
