File: hardware/06_protection.kicad_sch (KiCad schematic)
At the start: 216 parts, among them K601 TLP3545A, K602 TLP3545A, K603 TLP3545A, K604 TLP3545A, Q612 MMBT3904, Q614 MMBT3904, Q616 AO3400A, Q617 AO3400A, Q618 2N7002, Q619 AO3400A, Q620 AO3400A, Q621 2N7002, Q622 AO3400A, Q623 MMBT3904, Q624 MMBT3904, Q625 MMBT3904, Q626 MMBT3904, Q627 MMBT3904, U603 TLV1704, U604 OPA2333, U605 TLV3402, U606 TLV1704, U607 74AUP1G17, U608 74LVC1G74, U609 TLV1704, U610 TLV1704, U611 TLV1704, U612 TLV1704, U613 TLV3402, U614 TLV3402, U615 TLV3402, U616 TLV3402, U617 TLV3402, U618 TLV3402, U619 TLV3402, U620 TLV3402, U621 SN74AUP2G17DCKR

Commit message: feat: LCSC numbers for C631-C634 (C569856) and R402-R416 (C4101918)
Owner-supplied JLC numbers, checked against the JLCPCB part pages: both are
the exact MPNs (C4101918 is pre-order, 0 in stock). Applied as checked
overrides in generate_schematic.py; schematic, BOM and board LCSC fields
regenerated. X202/X203 stay open: C5122395 is a frequency-less NZ2520SDA
listing, and C2073999 (RR0816P-202-D, 0.5 %) was rejected.

Co-Authored-By: Claude Opus 5.5 <noreply@anthropic.com>
Parts:
- C631, C632, C633, C634: LCSC — -> C569856; LCSC Part # — -> C569856; Source Global sourcing -> JLCPCB C569856; order availability recheck
Changed lines of the file:
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@@
 (property "Datasheet" "" (at 187.96 171.45 0) (effects (font (size 1.016 1.016)) (hide yes)))
 (property "MPN" "Panasonic ECH-U1H224GX9" (at 187.96 171.45 0) (effects (font (size 1.016 1.016)) (hide yes)))
-(property "LCSC" "—" (at 187.96 171.45 0) (effects (font (size 1.016 1.016)) (hide yes)))
-(property "LCSC Part #" "—" (at 187.96 171.45 0) (effects (font (size 1.016 1.016)) (hide yes)))
+(property "LCSC" "C569856" (at 187.96 171.45 0) (effects (font (size 1.016 1.016)) (hide yes)))
+(property "LCSC Part #" "C569856" (at 187.96 171.45 0) (effects (font (size 1.016 1.016)) (hide yes)))
 (property "Assembly" "Yes" (at 187.96 171.45 0) (effects (font (size 1.016 1.016)) (hide yes)))
 (property "Package" "2416 (6041 metric), 6.0 × 4.1 × 2.8 mm (3.0 mm max)" (at 187.96 171.45 0) (effects (font (size 1.016 1.016)) (hide yes)))
 (property "Rating/Tolerance" "50 V DC PPS film ±2 % (G), TC bound ±0.5 % 0–60 °C; MSL 1" (at 187.96 171.45 0) (effects (font (size 1.016 1.016)) (hide yes)))
-(property "Source" "Global sourcing" (at 187.96 171.45 0) (effects (font (size 1.016 1.016)) (hide yes)))
+(property "Source" "JLCPCB C569856; order availability recheck" (at 187.96 171.45 0) (effects (font (size 1.016 1.016)) (hide yes)))
 (property "Workbook Value" "220 nF" (at 187.96 171.45 0) (effects (font (size 1.016 1.016)) (hide yes)))
 (property "Footprint status" "VERIFY G-3" (at 187.96 171.45 0) (effects (font (size 1.016 1.016)) (hide yes)))
@@
 (property "Datasheet" "" (at 233.68 171.45 0) (effects (font (size 1.016 1.016)) (hide yes)))
 (property "MPN" "Panasonic ECH-U1H224GX9" (at 233.68 171.45 0) (effects (font (size 1.016 1.016)) (hide yes)))
-(property "LCSC" "—" (at 233.68 171.45 0) (effects (font (size 1.016 1.016)) (hide yes)))
-(property "LCSC Part #" "—" (at 233.68 171.45 0) (effects (font (size 1.016 1.016)) (hide yes)))
+(property "LCSC" "C569856" (at 233.68 171.45 0) (effects (font (size 1.016 1.016)) (hide yes)))
+(property "LCSC Part #" "C569856" (at 233.68 171.45 0) (effects (font (size 1.016 1.016)) (hide yes)))
 (property "Assembly" "Yes" (at 233.68 171.45 0) (effects (font (size 1.016 1.016)) (hide yes)))
 (property "Package" "2416 (6041 metric), 6.0 × 4.1 × 2.8 mm (3.0 mm max)" (at 233.68 171.45 0) (effects (font (size 1.016 1.016)) (hide yes)))
 (property "Rating/Tolerance" "50 V DC PPS film ±2 % (G), TC bound ±0.5 % 0–60 °C; MSL 1" (at 233.68 171.45 0) (effects (font (size 1.016 1.016)) (hide yes)))
-(property "Source" "Global sourcing" (at 233.68 171.45 0) (effects (font (size 1.016 1.016)) (hide yes)))
+(property "Source" "JLCPCB C569856; order availability recheck" (at 233.68 171.45 0) (effects (font (size 1.016 1.016)) (hide yes)))
 (property "Workbook Value" "220 nF" (at 233.68 171.45 0) (effects (font (size 1.016 1.016)) (hide yes)))
 (property "Footprint status" "VERIFY G-3" (at 233.68 171.45 0) (effects (font (size 1.016 1.016)) (hide yes)))
@@
 (property "Datasheet" "" (at 279.4 171.45 0) (effects (font (size 1.016 1.016)) (hide yes)))
 (property "MPN" "Panasonic ECH-U1H224GX9" (at 279.4 171.45 0) (effects (font (size 1.016 1.016)) (hide yes)))
-(property "LCSC" "—" (at 279.4 171.45 0) (effects (font (size 1.016 1.016)) (hide yes)))
-(property "LCSC Part #" "—" (at 279.4 171.45 0) (effects (font (size 1.016 1.016)) (hide yes)))
+(property "LCSC" "C569856" (at 279.4 171.45 0) (effects (font (size 1.016 1.016)) (hide yes)))
+(property "LCSC Part #" "C569856" (at 279.4 171.45 0) (effects (font (size 1.016 1.016)) (hide yes)))
 (property "Assembly" "Yes" (at 279.4 171.45 0) (effects (font (size 1.016 1.016)) (hide yes)))
 (property "Package" "2416 (6041 metric), 6.0 × 4.1 × 2.8 mm (3.0 mm max)" (at 279.4 171.45 0) (effects (font (size 1.016 1.016)) (hide yes)))
 (property "Rating/Tolerance" "50 V DC PPS film ±2 % (G), TC bound ±0.5 % 0–60 °C; MSL 1" (at 279.4 171.45 0) (effects (font (size 1.016 1.016)) (hide yes)))
-(property "Source" "Global sourcing" (at 279.4 171.45 0) (effects (font (size 1.016 1.016)) (hide yes)))
+(property "Source" "JLCPCB C569856; order availability recheck" (at 279.4 171.45 0) (effects (font (size 1.016 1.016)) (hide yes)))
 (property "Workbook Value" "220 nF" (at 279.4 171.45 0) (effects (font (size 1.016 1.016)) (hide yes)))
 (property "Footprint status" "VERIFY G-3" (at 279.4 171.45 0) (effects (font (size 1.016 1.016)) (hide yes)))
@@
 (property "Datasheet" "" (at 325.12 171.45 0) (effects (font (size 1.016 1.016)) (hide yes)))
 (property "MPN" "Panasonic ECH-U1H224GX9" (at 325.12 171.45 0) (effects (font (size 1.016 1.016)) (hide yes)))
-(property "LCSC" "—" (at 325.12 171.45 0) (effects (font (size 1.016 1.016)) (hide yes)))
-(property "LCSC Part #" "—" (at 325.12 171.45 0) (effects (font (size 1.016 1.016)) (hide yes)))
+(property "LCSC" "C569856" (at 325.12 171.45 0) (effects (font (size 1.016 1.016)) (hide yes)))
+(property "LCSC Part #" "C569856" (at 325.12 171.45 0) (effects (font (size 1.016 1.016)) (hide yes)))
 (property "Assembly" "Yes" (at 325.12 171.45 0) (effects (font (size 1.016 1.016)) (hide yes)))
 (property "Package" "2416 (6041 metric), 6.0 × 4.1 × 2.8 mm (3.0 mm max)" (at 325.12 171.45 0) (effects (font (size 1.016 1.016)) (hide yes)))
 (property "Rating/Tolerance" "50 V DC PPS film ±2 % (G), TC bound ±0.5 % 0–60 °C; MSL 1" (at 325.12 171.45 0) (effects (font (size 1.016 1.016)) (hide yes)))
-(property "Source" "Global sourcing" (at 325.12 171.45 0) (effects (font (size 1.016 1.016)) (hide yes)))
+(property "Source" "JLCPCB C569856; order availability recheck" (at 325.12 171.45 0) (effects (font (size 1.016 1.016)) (hide yes)))
 (property "Workbook Value" "220 nF" (at 325.12 171.45 0) (effects (font (size 1.016 1.016)) (hide yes)))
 (property "Footprint status" "VERIFY G-3" (at 325.12 171.45 0) (effects (font (size 1.016 1.016)) (hide yes)))
