File: hardware/08_test_pads.kicad_sch (KiCad schematic)
At the start: 63 parts

Commit message: Recapture DAC-HPA schematic for design set v1.1
Parts:
- TP701, TP702, TP703, TP704, TP705, TP706, TP707, TP708, TP709, TP710, TP711, TP712, TP713, TP714, TP715, TP716, TP717, TP718, TP719, TP720, TP721, TP722, TP723, TP724, TP725, TP726, TP727, TP728, TP729, TP730, TP731, TP733, TP734, TP735, TP736, TP737, TP738, TP739, TP740, TP741, TP742, TP743, TP744, TP745, TP746, TP747, TP748, TP749, TP750, TP751, TP752, TP753: symbol DAC_HPA:P180 -> DAC_HPA:P183
