File: hardware/04_iv_output_legs.kicad_sch (KiCad schematic)
At the start: 83 parts, among them U401 OPA1622IDRCR, U402 OPA1622IDRCR, U403 OPA2210IDR, U404 OPA2210IDR

Commit message: Reassess DAC placement and add audio EMI geometry audit
Parts:
- U403, U404: value OPA2210IDR -> OPA2210IDGKR; footprint JLC_Imported:SOIC-8_L4.9-W3.9-P1.27-LS6.0-BL-2 -> JLC_Imported:VSSOP-8_L3.0-W3.0-P0.65-LS5.0-BL; LCSC C1849415 -> C2876414; LCSC Part # C1849415 -> C2876414; MPN TI OPA2210IDR -> TI OPA2210IDGKR; Package SOIC-8 -> VSSOP-8 (DGK); Source JLCPCB library -> JLCPCB Extended SMT (pre-order)
Changed lines of the file:
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@@
 (symbol (lib_id "DAC_HPA:P080") (at 184.15 67.31 0) (unit 1) (exclude_from_sim no) (in_bom yes) (on_board yes) (dnp no)
 (property "Reference" "U403" (at 184.15 58.42 0) (effects (font (size 0.889 0.889))))
-(property "Value" "OPA2210IDR" (at 184.15 76.2 0) (effects (font (size 0.889 0.889))))
-(property "Footprint" "JLC_Imported:SOIC-8_L4.9-W3.9-P1.27-LS6.0-BL-2" (at 184.15 67.31 0) (effects (font (size 1.016 1.016)) (hide yes)))
+(property "Value" "OPA2210IDGKR" (at 184.15 76.2 0) (effects (font (size 0.889 0.889))))
+(property "Footprint" "JLC_Imported:VSSOP-8_L3.0-W3.0-P0.65-LS5.0-BL" (at 184.15 67.31 0) (effects (font (size 1.016 1.016)) (hide yes)))
 (property "Datasheet" "https://www.ti.com/lit/ds/symlink/opa2210.pdf (SBOS924H)" (at 184.15 67.31 0) (effects (font (size 1.016 1.016)) (hide yes)))
-(property "MPN" "TI OPA2210IDR" (at 184.15 67.31 0) (effects (font (size 1.016 1.016)) (hide yes)))
-(property "LCSC" "C1849415" (at 184.15 67.31 0) (effects (font (size 1.016 1.016)) (hide yes)))
-(property "LCSC Part #" "C1849415" (at 184.15 67.31 0) (effects (font (size 1.016 1.016)) (hide yes)))
+(property "MPN" "TI OPA2210IDGKR" (at 184.15 67.31 0) (effects (font (size 1.016 1.016)) (hide yes)))
+(property "LCSC" "C2876414" (at 184.15 67.31 0) (effects (font (size 1.016 1.016)) (hide yes)))
+(property "LCSC Part #" "C2876414" (at 184.15 67.31 0) (effects (font (size 1.016 1.016)) (hide yes)))
 (property "Assembly" "Yes" (at 184.15 67.31 0) (effects (font (size 1.016 1.016)) (hide yes)))
-(property "Package" "SOIC-8" (at 184.15 67.31 0) (effects (font (size 1.016 1.016)) (hide yes)))
+(property "Package" "VSSOP-8 (DGK)" (at 184.15 67.31 0) (effects (font (size 1.016 1.016)) (hide yes)))
 (property "Rating/Tolerance" "Vos 35 µV, IQ 2.5 mA/ch max, CM (V-)+1.5…(V+)-1.5 V" (at 184.15 67.31 0) (effects (font (size 1.016 1.016)) (hide yes)))
-(property "Source" "JLCPCB library" (at 184.15 67.31 0) (effects (font (size 1.016 1.016)) (hide yes)))
+(property "Source" "JLCPCB Extended SMT (pre-order)" (at 184.15 67.31 0) (effects (font (size 1.016 1.016)) (hide yes)))
 (property "Workbook Value" "OPA2210IDR" (at 184.15 67.31 0) (effects (font (size 1.016 1.016)) (hide yes)))
 (property "Footprint status" "VERIFY G-3" (at 184.15 67.31 0) (effects (font (size 1.016 1.016)) (hide yes)))
@@
 (symbol (lib_id "DAC_HPA:P080") (at 242.57 67.31 0) (unit 1) (exclude_from_sim no) (in_bom yes) (on_board yes) (dnp no)
 (property "Reference" "U404" (at 242.57 58.42 0) (effects (font (size 0.889 0.889))))
-(property "Value" "OPA2210IDR" (at 242.57 76.2 0) (effects (font (size 0.889 0.889))))
-(property "Footprint" "JLC_Imported:SOIC-8_L4.9-W3.9-P1.27-LS6.0-BL-2" (at 242.57 67.31 0) (effects (font (size 1.016 1.016)) (hide yes)))
+(property "Value" "OPA2210IDGKR" (at 242.57 76.2 0) (effects (font (size 0.889 0.889))))
+(property "Footprint" "JLC_Imported:VSSOP-8_L3.0-W3.0-P0.65-LS5.0-BL" (at 242.57 67.31 0) (effects (font (size 1.016 1.016)) (hide yes)))
 (property "Datasheet" "https://www.ti.com/lit/ds/symlink/opa2210.pdf (SBOS924H)" (at 242.57 67.31 0) (effects (font (size 1.016 1.016)) (hide yes)))
-(property "MPN" "TI OPA2210IDR" (at 242.57 67.31 0) (effects (font (size 1.016 1.016)) (hide yes)))
-(property "LCSC" "C1849415" (at 242.57 67.31 0) (effects (font (size 1.016 1.016)) (hide yes)))
-(property "LCSC Part #" "C1849415" (at 242.57 67.31 0) (effects (font (size 1.016 1.016)) (hide yes)))
+(property "MPN" "TI OPA2210IDGKR" (at 242.57 67.31 0) (effects (font (size 1.016 1.016)) (hide yes)))
+(property "LCSC" "C2876414" (at 242.57 67.31 0) (effects (font (size 1.016 1.016)) (hide yes)))
+(property "LCSC Part #" "C2876414" (at 242.57 67.31 0) (effects (font (size 1.016 1.016)) (hide yes)))
 (property "Assembly" "Yes" (at 242.57 67.31 0) (effects (font (size 1.016 1.016)) (hide yes)))
-(property "Package" "SOIC-8" (at 242.57 67.31 0) (effects (font (size 1.016 1.016)) (hide yes)))
+(property "Package" "VSSOP-8 (DGK)" (at 242.57 67.31 0) (effects (font (size 1.016 1.016)) (hide yes)))
 (property "Rating/Tolerance" "Vos 35 µV, IQ 2.5 mA/ch max, CM (V-)+1.5…(V+)-1.5 V" (at 242.57 67.31 0) (effects (font (size 1.016 1.016)) (hide yes)))
-(property "Source" "JLCPCB library" (at 242.57 67.31 0) (effects (font (size 1.016 1.016)) (hide yes)))
+(property "Source" "JLCPCB Extended SMT (pre-order)" (at 242.57 67.31 0) (effects (font (size 1.016 1.016)) (hide yes)))
 (property "Workbook Value" "OPA2210IDR" (at 242.57 67.31 0) (effects (font (size 1.016 1.016)) (hide yes)))
 (property "Footprint status" "VERIFY G-3" (at 242.57 67.31 0) (effects (font (size 1.016 1.016)) (hide yes)))

Commit message: Route amplifier enables and audit low-DCR output-link ECO
Parts:
- R417, R418, R419, R420: LCSC C17168 -> C4044221; LCSC Part # C17168 -> C4044221; MPN UNI-ROYAL 0402WGF0000TCE -> YAGEO PA0402-R-070RL; Rating/Tolerance jumper, ≤ 50 mΩ -> jumper, ≤ 1 mΩ (manufacturer maximum); Source JLCPCB library -> JLCPCB Extended SMT; stock must be rechecked at order
Changed lines of the file:
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@@
 (property "Value" "0 Ω" (at 279.4 222.25 0) (effects (font (size 0.889 0.889))))
 (property "Footprint" "Resistor_SMD:R_0402_1005Metric" (at 279.4 217.17 0) (effects (font (size 1.016 1.016)) (hide yes)))
-(property "Datasheet" "https://www.lcsc.com/product-detail/C17168.html" (at 279.4 217.17 0) (effects (font (size 1.016 1.016)) (hide yes)))
-(property "MPN" "UNI-ROYAL 0402WGF0000TCE" (at 279.4 217.17 0) (effects (font (size 1.016 1.016)) (hide yes)))
-(property "LCSC" "C17168" (at 279.4 217.17 0) (effects (font (size 1.016 1.016)) (hide yes)))
-(property "LCSC Part #" "C17168" (at 279.4 217.17 0) (effects (font (size 1.016 1.016)) (hide yes)))
+(property "Datasheet" "https://www.yageogroup.com/content/Resource%20Library/Datasheet/PYU-PA_JUMPER_L_51_ROHS.pdf" (at 279.4 217.17 0) (effects (font (size 1.016 1.016)) (hide yes)))
+(property "MPN" "YAGEO PA0402-R-070RL" (at 279.4 217.17 0) (effects (font (size 1.016 1.016)) (hide yes)))
+(property "LCSC" "C4044221" (at 279.4 217.17 0) (effects (font (size 1.016 1.016)) (hide yes)))
+(property "LCSC Part #" "C4044221" (at 279.4 217.17 0) (effects (font (size 1.016 1.016)) (hide yes)))
 (property "Assembly" "Yes" (at 279.4 217.17 0) (effects (font (size 1.016 1.016)) (hide yes)))
 (property "Package" "0402" (at 279.4 217.17 0) (effects (font (size 1.016 1.016)) (hide yes)))
-(property "Rating/Tolerance" "jumper, ≤ 50 mΩ" (at 279.4 217.17 0) (effects (font (size 1.016 1.016)) (hide yes)))
-(property "Source" "JLCPCB library" (at 279.4 217.17 0) (effects (font (size 1.016 1.016)) (hide yes)))
+(property "Rating/Tolerance" "jumper, ≤ 1 mΩ (manufacturer maximum)" (at 279.4 217.17 0) (effects (font (size 1.016 1.016)) (hide yes)))
+(property "Source" "JLCPCB Extended SMT; stock must be rechecked at order" (at 279.4 217.17 0) (effects (font (size 1.016 1.016)) (hide yes)))
 (property "Workbook Value" "0 Ω" (at 279.4 217.17 0) (effects (font (size 1.016 1.016)) (hide yes)))
 (property "Footprint status" "VERIFY G-3" (at 279.4 217.17 0) (effects (font (size 1.016 1.016)) (hide yes)))
@@
 (property "Value" "0 Ω" (at 325.12 222.25 0) (effects (font (size 0.889 0.889))))
 (property "Footprint" "Resistor_SMD:R_0402_1005Metric" (at 325.12 217.17 0) (effects (font (size 1.016 1.016)) (hide yes)))
-(property "Datasheet" "https://www.lcsc.com/product-detail/C17168.html" (at 325.12 217.17 0) (effects (font (size 1.016 1.016)) (hide yes)))
-(property "MPN" "UNI-ROYAL 0402WGF0000TCE" (at 325.12 217.17 0) (effects (font (size 1.016 1.016)) (hide yes)))
-(property "LCSC" "C17168" (at 325.12 217.17 0) (effects (font (size 1.016 1.016)) (hide yes)))
-(property "LCSC Part #" "C17168" (at 325.12 217.17 0) (effects (font (size 1.016 1.016)) (hide yes)))
+(property "Datasheet" "https://www.yageogroup.com/content/Resource%20Library/Datasheet/PYU-PA_JUMPER_L_51_ROHS.pdf" (at 325.12 217.17 0) (effects (font (size 1.016 1.016)) (hide yes)))
+(property "MPN" "YAGEO PA0402-R-070RL" (at 325.12 217.17 0) (effects (font (size 1.016 1.016)) (hide yes)))
+(property "LCSC" "C4044221" (at 325.12 217.17 0) (effects (font (size 1.016 1.016)) (hide yes)))
+(property "LCSC Part #" "C4044221" (at 325.12 217.17 0) (effects (font (size 1.016 1.016)) (hide yes)))
 (property "Assembly" "Yes" (at 325.12 217.17 0) (effects (font (size 1.016 1.016)) (hide yes)))
 (property "Package" "0402" (at 325.12 217.17 0) (effects (font (size 1.016 1.016)) (hide yes)))
-(property "Rating/Tolerance" "jumper, ≤ 50 mΩ" (at 325.12 217.17 0) (effects (font (size 1.016 1.016)) (hide yes)))
-(property "Source" "JLCPCB library" (at 325.12 217.17 0) (effects (font (size 1.016 1.016)) (hide yes)))
+(property "Rating/Tolerance" "jumper, ≤ 1 mΩ (manufacturer maximum)" (at 325.12 217.17 0) (effects (font (size 1.016 1.016)) (hide yes)))
+(property "Source" "JLCPCB Extended SMT; stock must be rechecked at order" (at 325.12 217.17 0) (effects (font (size 1.016 1.016)) (hide yes)))
 (property "Workbook Value" "0 Ω" (at 325.12 217.17 0) (effects (font (size 1.016 1.016)) (hide yes)))
 (property "Footprint status" "VERIFY G-3" (at 325.12 217.17 0) (effects (font (size 1.016 1.016)) (hide yes)))
@@
 (property "Value" "0 Ω" (at 370.84 222.25 0) (effects (font (size 0.889 0.889))))
 (property "Footprint" "Resistor_SMD:R_0402_1005Metric" (at 370.84 217.17 0) (effects (font (size 1.016 1.016)) (hide yes)))
-(property "Datasheet" "https://www.lcsc.com/product-detail/C17168.html" (at 370.84 217.17 0) (effects (font (size 1.016 1.016)) (hide yes)))
-(property "MPN" "UNI-ROYAL 0402WGF0000TCE" (at 370.84 217.17 0) (effects (font (size 1.016 1.016)) (hide yes)))
-(property "LCSC" "C17168" (at 370.84 217.17 0) (effects (font (size 1.016 1.016)) (hide yes)))
-(property "LCSC Part #" "C17168" (at 370.84 217.17 0) (effects (font (size 1.016 1.016)) (hide yes)))
+(property "Datasheet" "https://www.yageogroup.com/content/Resource%20Library/Datasheet/PYU-PA_JUMPER_L_51_ROHS.pdf" (at 370.84 217.17 0) (effects (font (size 1.016 1.016)) (hide yes)))
+(property "MPN" "YAGEO PA0402-R-070RL" (at 370.84 217.17 0) (effects (font (size 1.016 1.016)) (hide yes)))
+(property "LCSC" "C4044221" (at 370.84 217.17 0) (effects (font (size 1.016 1.016)) (hide yes)))
+(property "LCSC Part #" "C4044221" (at 370.84 217.17 0) (effects (font (size 1.016 1.016)) (hide yes)))
 (property "Assembly" "Yes" (at 370.84 217.17 0) (effects (font (size 1.016 1.016)) (hide yes)))
 (property "Package" "0402" (at 370.84 217.17 0) (effects (font (size 1.016 1.016)) (hide yes)))
-(property "Rating/Tolerance" "jumper, ≤ 50 mΩ" (at 370.84 217.17 0) (effects (font (size 1.016 1.016)) (hide yes)))
-(property "Source" "JLCPCB library" (at 370.84 217.17 0) (effects (font (size 1.016 1.016)) (hide yes)))
+(property "Rating/Tolerance" "jumper, ≤ 1 mΩ (manufacturer maximum)" (at 370.84 217.17 0) (effects (font (size 1.016 1.016)) (hide yes)))
+(property "Source" "JLCPCB Extended SMT; stock must be rechecked at order" (at 370.84 217.17 0) (effects (font (size 1.016 1.016)) (hide yes)))
 (property "Workbook Value" "0 Ω" (at 370.84 217.17 0) (effects (font (size 1.016 1.016)) (hide yes)))
 (property "Footprint status" "VERIFY G-3" (at 370.84 217.17 0) (effects (font (size 1.016 1.016)) (hide yes)))
@@
 (property "Value" "0 Ω" (at 50.8 237.49 0) (effects (font (size 0.889 0.889))))
 (property "Footprint" "Resistor_SMD:R_0402_1005Metric" (at 50.8 232.41 0) (effects (font (size 1.016 1.016)) (hide yes)))
-(property "Datasheet" "https://www.lcsc.com/product-detail/C17168.html" (at 50.8 232.41 0) (effects (font (size 1.016 1.016)) (hide yes)))
-(property "MPN" "UNI-ROYAL 0402WGF0000TCE" (at 50.8 232.41 0) (effects (font (size 1.016 1.016)) (hide yes)))
-(property "LCSC" "C17168" (at 50.8 232.41 0) (effects (font (size 1.016 1.016)) (hide yes)))
-(property "LCSC Part #" "C17168" (at 50.8 232.41 0) (effects (font (size 1.016 1.016)) (hide yes)))
+(property "Datasheet" "https://www.yageogroup.com/content/Resource%20Library/Datasheet/PYU-PA_JUMPER_L_51_ROHS.pdf" (at 50.8 232.41 0) (effects (font (size 1.016 1.016)) (hide yes)))
+(property "MPN" "YAGEO PA0402-R-070RL" (at 50.8 232.41 0) (effects (font (size 1.016 1.016)) (hide yes)))
+(property "LCSC" "C4044221" (at 50.8 232.41 0) (effects (font (size 1.016 1.016)) (hide yes)))
+(property "LCSC Part #" "C4044221" (at 50.8 232.41 0) (effects (font (size 1.016 1.016)) (hide yes)))
 (property "Assembly" "Yes" (at 50.8 232.41 0) (effects (font (size 1.016 1.016)) (hide yes)))
 (property "Package" "0402" (at 50.8 232.41 0) (effects (font (size 1.016 1.016)) (hide yes)))
-(property "Rating/Tolerance" "jumper, ≤ 50 mΩ" (at 50.8 232.41 0) (effects (font (size 1.016 1.016)) (hide yes)))
-(property "Source" "JLCPCB library" (at 50.8 232.41 0) (effects (font (size 1.016 1.016)) (hide yes)))
+(property "Rating/Tolerance" "jumper, ≤ 1 mΩ (manufacturer maximum)" (at 50.8 232.41 0) (effects (font (size 1.016 1.016)) (hide yes)))
+(property "Source" "JLCPCB Extended SMT; stock must be rechecked at order" (at 50.8 232.41 0) (effects (font (size 1.016 1.016)) (hide yes)))
 (property "Workbook Value" "0 Ω" (at 50.8 232.41 0) (effects (font (size 1.016 1.016)) (hide yes)))
 (property "Footprint status" "VERIFY G-3" (at 50.8 232.41 0) (effects (font (size 1.016 1.016)) (hide yes)))

Commit message: Route manual DAC I/V and U501 macros with chamfered copper
Connections:
- net DACL: now also U403.6 (-IN B); no longer U403.2 (-IN A)
- net DACLB: now also U403.2 (-IN A); no longer U403.6 (-IN B)
- net DACR: now also U404.6 (-IN B); no longer U404.2 (-IN A)
- net DACRB: now also U404.2 (-IN A); no longer U404.6 (-IN B)
- net N4_IVL_N: now also U403.1 (OUT A); no longer U403.7 (OUT B)
- net N4_IVL_P: now also U403.7 (OUT B); no longer U403.1 (OUT A)
- net N4_IVR_N: now also U404.1 (OUT A); no longer U404.7 (OUT B)
- net N4_IVR_P: now also U404.7 (OUT B); no longer U404.1 (OUT A)
Changed lines of the file:
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@@
 )
 (wire (pts (xy 168.91 63.5) (xy 166.37 63.5)) (stroke (width 0) (type solid)))
-(global_label "N4_IVL_P" (shape bidirectional) (at 166.37 63.5 180) (effects (font (size 0.762 0.762)) (justify right bottom)))
+(global_label "N4_IVL_N" (shape bidirectional) (at 166.37 63.5 180) (effects (font (size 0.762 0.762)) (justify right bottom)))
 (wire (pts (xy 168.91 66.04) (xy 166.37 66.04)) (stroke (width 0) (type solid)))
-(global_label "DACL" (shape bidirectional) (at 166.37 66.04 180) (effects (font (size 0.762 0.762)) (justify right bottom)))
+(global_label "DACLB" (shape bidirectional) (at 166.37 66.04 180) (effects (font (size 0.762 0.762)) (justify right bottom)))
 (wire (pts (xy 168.91 68.58) (xy 166.37 68.58)) (stroke (width 0) (type solid)))
 (global_label "VREF" (shape bidirectional) (at 166.37 68.58 180) (effects (font (size 0.762 0.762)) (justify right bottom)))
@@
 (global_label "VREF" (shape bidirectional) (at 201.93 63.5 0) (effects (font (size 0.762 0.762)) (justify left bottom)))
 (wire (pts (xy 199.39 66.04) (xy 201.93 66.04)) (stroke (width 0) (type solid)))
-(global_label "DACLB" (shape bidirectional) (at 201.93 66.04 0) (effects (font (size 0.762 0.762)) (justify left bottom)))
+(global_label "DACL" (shape bidirectional) (at 201.93 66.04 0) (effects (font (size 0.762 0.762)) (justify left bottom)))
 (wire (pts (xy 199.39 68.58) (xy 201.93 68.58)) (stroke (width 0) (type solid)))
-(global_label "N4_IVL_N" (shape bidirectional) (at 201.93 68.58 0) (effects (font (size 0.762 0.762)) (justify left bottom)))
+(global_label "N4_IVL_P" (shape bidirectional) (at 201.93 68.58 0) (effects (font (size 0.762 0.762)) (justify left bottom)))
 (wire (pts (xy 199.39 71.12) (xy 201.93 71.12)) (stroke (width 0) (type solid)))
 (global_label "N4_VPOS_IV" (shape bidirectional) (at 201.93 71.12 0) (effects (font (size 0.762 0.762)) (justify left bottom)))
@@
 )
 (wire (pts (xy 227.33 63.5) (xy 224.79 63.5)) (stroke (width 0) (type solid)))
-(global_label "N4_IVR_P" (shape bidirectional) (at 224.79 63.5 180) (effects (font (size 0.762 0.762)) (justify right bottom)))
+(global_label "N4_IVR_N" (shape bidirectional) (at 224.79 63.5 180) (effects (font (size 0.762 0.762)) (justify right bottom)))
 (wire (pts (xy 227.33 66.04) (xy 224.79 66.04)) (stroke (width 0) (type solid)))
-(global_label "DACR" (shape bidirectional) (at 224.79 66.04 180) (effects (font (size 0.762 0.762)) (justify right bottom)))
+(global_label "DACRB" (shape bidirectional) (at 224.79 66.04 180) (effects (font (size 0.762 0.762)) (justify right bottom)))
 (wire (pts (xy 227.33 68.58) (xy 224.79 68.58)) (stroke (width 0) (type solid)))
 (global_label "VREF" (shape bidirectional) (at 224.79 68.58 180) (effects (font (size 0.762 0.762)) (justify right bottom)))
@@
 (global_label "VREF" (shape bidirectional) (at 260.35 63.5 0) (effects (font (size 0.762 0.762)) (justify left bottom)))
 (wire (pts (xy 257.81 66.04) (xy 260.35 66.04)) (stroke (width 0) (type solid)))
-(global_label "DACRB" (shape bidirectional) (at 260.35 66.04 0) (effects (font (size 0.762 0.762)) (justify left bottom)))
+(global_label "DACR" (shape bidirectional) (at 260.35 66.04 0) (effects (font (size 0.762 0.762)) (justify left bottom)))
 (wire (pts (xy 257.81 68.58) (xy 260.35 68.58)) (stroke (width 0) (type solid)))
-(global_label "N4_IVR_N" (shape bidirectional) (at 260.35 68.58 0) (effects (font (size 0.762 0.762)) (justify left bottom)))
+(global_label "N4_IVR_P" (shape bidirectional) (at 260.35 68.58 0) (effects (font (size 0.762 0.762)) (justify left bottom)))
 (wire (pts (xy 257.81 71.12) (xy 260.35 71.12)) (stroke (width 0) (type solid)))
 (global_label "N4_VPOS_IV" (shape bidirectional) (at 260.35 71.12 0) (effects (font (size 0.762 0.762)) (justify left bottom)))
