File: hardware/04_iv_output_legs.kicad_sch (KiCad schematic)
At the start: 83 parts, among them U401 OPA1622IDRCR, U402 OPA1622IDRCR, U403 OPA2210IDGKR, U404 OPA2210IDGKR

Commit message: feat: ECO F10 ground-sense reference for the 3.5 mm output (owner-approved)
MATLAB sign-off found USB frame-rate digital ground current reaching the
single-ended output only ~1 dB below audibility on a 135 dB SPL/V IEM: the
difference-stage reference resistors R404/R408/R412/R416 tied to the plane
near the DAC, 45 mm from the J702 sleeve. They now return through the new
net N4_GSENSE to R448 (0 ohm, R107's part) at the J702 sleeve, which has a
dedicated Kelvin track to J702.1. Ground currents between the DAC area and
the jack become common mode for the difference stage instead of adding 1:1.

- Schematic: F10 overlay + R448 (535 parts, 253 nets); verifier deltas,
  notes and assembly counts updated; ERC 0.
- Layout: R448 above J702 (JLC edge spacing, jack access rule met); sense
  routed pair-first (R404-R408, R412-R416) then one L4 trunk to R448.
  Builder gains added_footprints (copy of an existing board footprint).
- Checks: frozen boards skip the F10 refs; integrated checker asserts the
  ground-sense topology. DRC 0, unconnected 0, VALIDATE_OK.

Co-Authored-By: Claude Opus 5.5 <noreply@anthropic.com>
Parts:
- added R448: 0 Ω, Resistor_SMD:R_0402_1005Metric, symbol DAC_HPA:P9006
Connections:
- net GND: now also R448.2; no longer R404.2, R408.2, R412.2, R416.2
- new net N4_GSENSE: R404.2, R408.2, R412.2, R416.2, R448.1
Changed lines of the file:
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@@
 (global_label "N4_LP_INP" (shape bidirectional) (at 43.18 201.93 180) (effects (font (size 0.762 0.762)) (justify right bottom)))
 (wire (pts (xy 55.88 201.93) (xy 58.42 201.93)) (stroke (width 0) (type solid)))
-(global_label "GND" (shape bidirectional) (at 58.42 201.93 0) (effects (font (size 0.762 0.762)) (justify left bottom)))
+(global_label "N4_GSENSE" (shape bidirectional) (at 58.42 201.93 0) (effects (font (size 0.762 0.762)) (justify left bottom)))
 (symbol (lib_id "DAC_HPA:P071") (at 96.52 201.93 0) (unit 1) (exclude_from_sim no) (in_bom yes) (on_board yes) (dnp no)
 (property "Reference" "R405" (at 96.52 196.85 0) (effects (font (size 0.889 0.889))))
@@
 (global_label "N4_LN_INP" (shape bidirectional) (at 226.06 201.93 180) (effects (font (size 0.762 0.762)) (justify right bottom)))
 (wire (pts (xy 238.76 201.93) (xy 241.3 201.93)) (stroke (width 0) (type solid)))
-(global_label "GND" (shape bidirectional) (at 241.3 201.93 0) (effects (font (size 0.762 0.762)) (justify left bottom)))
+(global_label "N4_GSENSE" (shape bidirectional) (at 241.3 201.93 0) (effects (font (size 0.762 0.762)) (justify left bottom)))
 (symbol (lib_id "DAC_HPA:P071") (at 279.4 201.93 0) (unit 1) (exclude_from_sim no) (in_bom yes) (on_board yes) (dnp no)
 (property "Reference" "R409" (at 279.4 196.85 0) (effects (font (size 0.889 0.889))))
@@
 (global_label "N4_RP_INP" (shape bidirectional) (at 43.18 217.17 180) (effects (font (size 0.762 0.762)) (justify right bottom)))
 (wire (pts (xy 55.88 217.17) (xy 58.42 217.17)) (stroke (width 0) (type solid)))
-(global_label "GND" (shape bidirectional) (at 58.42 217.17 0) (effects (font (size 0.762 0.762)) (justify left bottom)))
+(global_label "N4_GSENSE" (shape bidirectional) (at 58.42 217.17 0) (effects (font (size 0.762 0.762)) (justify left bottom)))
 (symbol (lib_id "DAC_HPA:P071") (at 96.52 217.17 0) (unit 1) (exclude_from_sim no) (in_bom yes) (on_board yes) (dnp no)
 (property "Reference" "R413" (at 96.52 212.09 0) (effects (font (size 0.889 0.889))))
@@
 (global_label "N4_RN_INP" (shape bidirectional) (at 226.06 217.17 180) (effects (font (size 0.762 0.762)) (justify right bottom)))
 (wire (pts (xy 238.76 217.17) (xy 241.3 217.17)) (stroke (width 0) (type solid)))
-(global_label "GND" (shape bidirectional) (at 241.3 217.17 0) (effects (font (size 0.762 0.762)) (justify left bottom)))
+(global_label "N4_GSENSE" (shape bidirectional) (at 241.3 217.17 0) (effects (font (size 0.762 0.762)) (justify left bottom)))
 (symbol (lib_id "DAC_HPA:P073") (at 279.4 217.17 0) (unit 1) (exclude_from_sim no) (in_bom yes) (on_board yes) (dnp no)
 (property "Reference" "R417" (at 279.4 212.09 0) (effects (font (size 0.889 0.889))))
@@
 (wire (pts (xy 55.88 262.89) (xy 58.42 262.89)) (stroke (width 0) (type solid)))
 (global_label "GND" (shape bidirectional) (at 58.42 262.89 0) (effects (font (size 0.762 0.762)) (justify left bottom)))
+(symbol (lib_id "DAC_HPA:P9006") (at 96.52 262.89 0) (unit 1) (exclude_from_sim no) (in_bom yes) (on_board yes) (dnp no)
+(property "Reference" "R448" (at 96.52 257.81 0) (effects (font (size 0.889 0.889))))
+(property "Value" "0 Ω" (at 96.52 267.97 0) (effects (font (size 0.889 0.889))))
+(property "Footprint" "Resistor_SMD:R_0402_1005Metric" (at 96.52 262.89 0) (effects (font (size 1.016 1.016)) (hide yes)))
+(property "Datasheet" "https://www.lcsc.com/product-detail/C17168.html" (at 96.52 262.89 0) (effects (font (size 1.016 1.016)) (hide yes)))
+(property "MPN" "UNI-ROYAL 0402WGF0000TCE" (at 96.52 262.89 0) (effects (font (size 1.016 1.016)) (hide yes)))
+(property "LCSC" "C17168" (at 96.52 262.89 0) (effects (font (size 1.016 1.016)) (hide yes)))
+(property "LCSC Part #" "C17168" (at 96.52 262.89 0) (effects (font (size 1.016 1.016)) (hide yes)))
+(property "Assembly" "Yes" (at 96.52 262.89 0) (effects (font (size 1.016 1.016)) (hide yes)))
+(property "Package" "0402" (at 96.52 262.89 0) (effects (font (size 1.016 1.016)) (hide yes)))
+(property "Rating/Tolerance" "jumper" (at 96.52 262.89 0) (effects (font (size 1.016 1.016)) (hide yes)))
+(property "Source" "JLCPCB library" (at 96.52 262.89 0) (effects (font (size 1.016 1.016)) (hide yes)))
+(property "Workbook Value" "— (functional ECO; absent from Parts List v0.9)" (at 96.52 262.89 0) (effects (font (size 1.016 1.016)) (hide yes)))
+(property "Footprint status" "VERIFY G-3" (at 96.52 262.89 0) (effects (font (size 1.016 1.016)) (hide yes)))
+(pin "1")
+(pin "2")
+(instances (project "DAC_HPA" (path "/0c6c0976-e401-5c8a-8977-bc60da031e5e/df299358-b873-5680-a36b-db04bd1b9572" (reference "R448") (unit 1))))
+)
+(wire (pts (xy 91.44 262.89) (xy 88.9 262.89)) (stroke (width 0) (type solid)))
+(global_label "N4_GSENSE" (shape bidirectional) (at 88.9 262.89 180) (effects (font (size 0.762 0.762)) (justify right bottom)))
+(wire (pts (xy 101.6 262.89) (xy 104.14 262.89)) (stroke (width 0) (type solid)))
+(global_label "GND" (shape bidirectional) (at 104.14 262.89 0) (effects (font (size 0.762 0.762)) (justify left bottom)))
 (symbol (lib_id "DAC_HPA:P079") (at 59.69 69.85 0) (unit 1) (exclude_from_sim no) (in_bom yes) (on_board yes) (dnp no)
 (property "Reference" "U401" (at 59.69 58.42 0) (effects (font (size 0.889 0.889))))

Commit message: feat: LCSC numbers for C631-C634 (C569856) and R402-R416 (C4101918)
Owner-supplied JLC numbers, checked against the JLCPCB part pages: both are
the exact MPNs (C4101918 is pre-order, 0 in stock). Applied as checked
overrides in generate_schematic.py; schematic, BOM and board LCSC fields
regenerated. X202/X203 stay open: C5122395 is a frequency-less NZ2520SDA
listing, and C2073999 (RR0816P-202-D, 0.5 %) was rejected.

Co-Authored-By: Claude Opus 5.5 <noreply@anthropic.com>
Parts:
- R402, R404, R406, R408, R410, R412, R414, R416: LCSC — -> C4101918; LCSC Part # — -> C4101918; Source Global sourcing -> JLCPCB C4101918 (pre-order, 0 stock on 19 Oct 2026)
