File: hardware/DAC_HPA_120x100_OUTPUT_MACRO_STUDY_ONLY.kicad_pcb (KiCad board)
At the start: 4 copper layers, 120 x 100 mm, 544 parts, among them J101 GCT USB4105-GF-A, J201 PCB pads (no component), J202 PCB pads (no component), J701 G-Switch GT-3321667P-01, J702 HRO PJ-332A-6A, K601 TLP3545A, K602 TLP3545A, K603 TLP3545A, K604 TLP3545A, Q207 AO3400A, Q502 AO3400A, Q503 AO3400A, Q504 AO3400A, Q505 AO3400A, Q506 AO3400A, Q507 MMBT3904, Q612 MMBT3904, Q614 MMBT3904, Q616 AO3400A, Q617 AO3400A, Q618 2N7002, Q619 AO3400A, Q620 AO3400A, Q621 2N7002, Q622 AO3400A, Q623 MMBT3904, Q624 MMBT3904, Q625 MMBT3904, Q626 MMBT3904, Q627 MMBT3904, U101 ST USBLC6-2SC6, U102 TI TPS25200DRVR, U103 TI TPD2E2U06DRLR, U201 CH32V307RCT6, U202 AGRV2KQ32, U205 74LVC1G157, U206 74LVC1G11, U208 74LVC3G34, U301 ES9018K2M, U302 3.3 V, 250 mA, U303 1.300 V (R533/R534), U401 OPA1622IDRCR, U402 OPA1622IDRCR, U403 OPA2210IDGKR, U404 OPA2210IDGKR, U501 +3.85 / -3.72 V, U502 3.3 V, 150 mA, U503 TI TPS259621DDAR, U504 3.3 V, 1 A, U505 TI TMUX1101DBVR, U603 TLV1704, U604 OPA2333, U605 TLV3402, U606 TLV1704, U607 74AUP1G17, U608 74LVC1G74, U609 TLV1704, U610 TLV1704, U611 TLV1704, U612 TLV1704, U613 TLV3402, U614 TLV3402, U615 TLV3402, U616 TLV3402, U617 TLV3402, U618 TLV3402, U619 TLV3402, U620 TLV3402, U621 SN74AUP2G17DCKR, X201 80.000 MHz, X202 49.152 MHz, X203 45.1584 MHz, Y201 8 MHz

Commit message: Add manually routed four-channel output macro study
Parts:
- moved R417 29.2 mm to (132.0, 97.2)
- moved R420 24.6 mm to (144.2, 68.9)
- moved C405 23.9 mm to (134.2, 76.5), turned to -90 degrees
- moved C407 21.2 mm to (134.2, 81.5), turned to 90 degrees
- moved R418 19.1 mm to (129.4, 64.9)
- moved R414 17.3 mm to (132.5, 81.5)
- moved C415 16.8 mm to (128.0, 93.5)
- moved R419 15.0 mm to (144.0, 83.4)
- moved R407 14.9 mm to (112.5, 84.5)
- moved C433 14.8 mm to (109.0, 84.0)
- moved C435 11.6 mm to (130.0, 73.0)
- moved U402 10.5 mm to (129.0, 79.0), turned to -90 degrees
- moved C434 10.0 mm to (112.5, 80.0)
- moved R402 9.30 mm to (120.5, 76.5), turned to -90 degrees
- moved C402 9.06 mm to (113.0, 78.0)
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Routing:
- net N4_LP_OUT: track 0.00 -> 30.7 mm, vias 0 -> 2
- net N4_RN_OUT: track 0.00 -> 27.6 mm, vias 0 -> 2
- net N4_LN_OUT: track 0.00 -> 24.3 mm, vias 0 -> 2
- net N4_RP_OUT: track 0.00 -> 23.7 mm
- net LEG_RP: track 0.00 -> 19.0 mm
- net LEG_RN: track 0.00 -> 6.31 mm
- net N4_RP_INN: track 0.00 -> 5.00 mm
- net N4_RN_INN: track 0.00 -> 5.00 mm
- net N4_LP_INN: track 0.00 -> 5.00 mm
- net N4_LN_INN: track 0.00 -> 5.00 mm
- net LEG_LP: track 0.00 -> 4.95 mm
- net LEG_LN: track 0.00 -> 4.55 mm
Other:
- board text added: "OUTPUT MACRO / MANUAL ROUTE STUDY — NO PCBA RELEASE"
- board text removed: "FUNCTIONAL ECO / MANUAL PLACEMENT — REVIEW ONLY"

Commit message: Route manual DAC I/V and U501 macros with chamfered copper
Connections:
- U403 pad 1: N4_IVL_P -> N4_IVL_N
- U403 pad 2: DACL -> DACLB
- U403 pad 6: DACLB -> DACL
- U403 pad 7: N4_IVL_N -> N4_IVL_P
- U404 pad 1: N4_IVR_P -> N4_IVR_N
- U404 pad 2: DACR -> DACRB
- U404 pad 6: DACRB -> DACR
- U404 pad 7: N4_IVR_N -> N4_IVR_P
