File: hardware/02_usb_bridge.kicad_sch (KiCad schematic)
At the start: 73 parts, among them J201 PCB pads (no component), J202 PCB pads (no component), Q207 AO3400A, U201 CH32V307RCT6, U202 AGRV2KQ32, U205 74LVC1G157, U206 74LVC1G11, U208 74LVC3G34, X201 80.000 MHz, X202 49.152 MHz, X203 45.1584 MHz, Y201 8 MHz

Commit message: feat: fit JLC SMD programming headers on J201 (MCU) and J202 (CPLD)
ECO F05: XKB X6511WVS-08H-C60D48R1 (C2883805) and X6511WVS-05H-C60D48R1
(C2883802) 2.54 mm SMD vertical headers replace the bare debug pad rows.
SMD keeps L2 whole and the inner-layer routes under the north edge intact.
Pin line moved 0.5 mm south for edge clearance; R241 and FID5 re-placed.
The replay gains a swapped_footprints manifest entry. Schematic CI steps
and VALIDATE_OK pass; 64 ratsnest links, 0 DRC.

Co-Authored-By: Claude Opus 5.5 <noreply@anthropic.com>
Parts:
- J201: value PCB pads (no component) -> X6511WVS-08H-C60D48R1; footprint DAC_HPA:J201_8_DebugPads_P2.54mm -> DAC_HPA:PinHeader_1x08_P2.54mm_SMD_XKB_X6511WVS-08H-C60D48R1; Assembly Pads -> Yes; LCSC — -> C2883805; LCSC Part # — -> C2883805; MPN PCB pads (no component) -> XKB X6511WVS-08H-C60D48R1; Package 8 SMD pads -> SMD 1x8 P2.54 mm vertical, staggered legs; Rating/Tolerance — -> 3 A, 250 V; 2.5 mm body, 6.0 mm mating pin; Source PCB copper -> JLCPCB C2883805; order availability recheck; Workbook Value — -> X6511WVS-08H-C60D48R1; now in the parts list
- J202: value PCB pads (no component) -> X6511WVS-05H-C60D48R1; footprint DAC_HPA:J202_5_JTAGPads_P2.54mm -> DAC_HPA:PinHeader_1x05_P2.54mm_SMD_XKB_X6511WVS-05H-C60D48R1; Assembly Pads -> Yes; LCSC — -> C2883802; LCSC Part # — -> C2883802; MPN PCB pads (no component) -> XKB X6511WVS-05H-C60D48R1; Package 5 SMD pads -> SMD 1x5 P2.54 mm vertical, staggered legs; Rating/Tolerance — -> 3 A, 250 V; 2.5 mm body, 6.0 mm mating pin; Source PCB copper -> JLCPCB C2883802; order availability recheck; Workbook Value — -> X6511WVS-05H-C60D48R1; now in the parts list
Changed lines of the file:
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@@
 (wire (pts (xy 147.32 262.89) (xy 149.86 262.89)) (stroke (width 0) (type solid)))
 (global_label "N2_V33_CPLD" (shape bidirectional) (at 149.86 262.89 0) (effects (font (size 0.762 0.762)) (justify left bottom)))
-(symbol (lib_id "DAC_HPA:P026") (at 215.9 67.31 0) (unit 1) (exclude_from_sim no) (in_bom no) (on_board yes) (dnp no)
+(symbol (lib_id "DAC_HPA:P026") (at 215.9 67.31 0) (unit 1) (exclude_from_sim no) (in_bom yes) (on_board yes) (dnp no)
 (property "Reference" "J201" (at 215.9 58.42 0) (effects (font (size 0.889 0.889))))
-(property "Value" "PCB pads (no component)" (at 215.9 76.2 0) (effects (font (size 0.889 0.889))))
-(property "Footprint" "DAC_HPA:J201_8_DebugPads_P2.54mm" (at 215.9 67.31 0) (effects (font (size 1.016 1.016)) (hide yes)))
-(property "Datasheet" "" (at 215.9 67.31 0) (effects (font (size 1.016 1.016)) (hide yes)))
-(property "MPN" "PCB pads (no component)" (at 215.9 67.31 0) (effects (font (size 1.016 1.016)) (hide yes)))
-(property "LCSC" "—" (at 215.9 67.31 0) (effects (font (size 1.016 1.016)) (hide yes)))
-(property "LCSC Part #" "—" (at 215.9 67.31 0) (effects (font (size 1.016 1.016)) (hide yes)))
-(property "Assembly" "Pads" (at 215.9 67.31 0) (effects (font (size 1.016 1.016)) (hide yes)))
-(property "Package" "8 SMD pads" (at 215.9 67.31 0) (effects (font (size 1.016 1.016)) (hide yes)))
-(property "Rating/Tolerance" "—" (at 215.9 67.31 0) (effects (font (size 1.016 1.016)) (hide yes)))
-(property "Source" "PCB copper" (at 215.9 67.31 0) (effects (font (size 1.016 1.016)) (hide yes)))
-(property "Workbook Value" "—" (at 215.9 67.31 0) (effects (font (size 1.016 1.016)) (hide yes)))
+(property "Value" "X6511WVS-08H-C60D48R1" (at 215.9 76.2 0) (effects (font (size 0.889 0.889))))
+(property "Footprint" "DAC_HPA:PinHeader_1x08_P2.54mm_SMD_XKB_X6511WVS-08H-C60D48R1" (at 215.9 67.31 0) (effects (font (size 1.016 1.016)) (hide yes)))
+(property "Datasheet" "https://www.lcsc.com/datasheet/C2883805.pdf" (at 215.9 67.31 0) (effects (font (size 1.016 1.016)) (hide yes)))
+(property "MPN" "XKB X6511WVS-08H-C60D48R1" (at 215.9 67.31 0) (effects (font (size 1.016 1.016)) (hide yes)))
+(property "LCSC" "C2883805" (at 215.9 67.31 0) (effects (font (size 1.016 1.016)) (hide yes)))
+(property "LCSC Part #" "C2883805" (at 215.9 67.31 0) (effects (font (size 1.016 1.016)) (hide yes)))
+(property "Assembly" "Yes" (at 215.9 67.31 0) (effects (font (size 1.016 1.016)) (hide yes)))
+(property "Package" "SMD 1x8 P2.54 mm vertical, staggered legs" (at 215.9 67.31 0) (effects (font (size 1.016 1.016)) (hide yes)))
+(property "Rating/Tolerance" "3 A, 250 V; 2.5 mm body, 6.0 mm mating pin" (at 215.9 67.31 0) (effects (font (size 1.016 1.016)) (hide yes)))
+(property "Source" "JLCPCB C2883805; order availability recheck" (at 215.9 67.31 0) (effects (font (size 1.016 1.016)) (hide yes)))
+(property "Workbook Value" "X6511WVS-08H-C60D48R1" (at 215.9 67.31 0) (effects (font (size 1.016 1.016)) (hide yes)))
 (property "Footprint status" "VERIFY G-3" (at 215.9 67.31 0) (effects (font (size 1.016 1.016)) (hide yes)))
 (pin "1")
@@
 (wire (pts (xy 232.41 71.12) (xy 234.95 71.12)) (stroke (width 0) (type solid)))
 (global_label "USART_RX" (shape bidirectional) (at 234.95 71.12 0) (effects (font (size 0.762 0.762)) (justify left bottom)))
-(symbol (lib_id "DAC_HPA:P027") (at 118.11 165.1 0) (unit 1) (exclude_from_sim no) (in_bom no) (on_board yes) (dnp no)
+(symbol (lib_id "DAC_HPA:P027") (at 118.11 165.1 0) (unit 1) (exclude_from_sim no) (in_bom yes) (on_board yes) (dnp no)
 (property "Reference" "J202" (at 118.11 157.48 0) (effects (font (size 0.889 0.889))))
-(property "Value" "PCB pads (no component)" (at 118.11 172.72 0) (effects (font (size 0.889 0.889))))
-(property "Footprint" "DAC_HPA:J202_5_JTAGPads_P2.54mm" (at 118.11 165.1 0) (effects (font (size 1.016 1.016)) (hide yes)))
-(property "Datasheet" "" (at 118.11 165.1 0) (effects (font (size 1.016 1.016)) (hide yes)))
-(property "MPN" "PCB pads (no component)" (at 118.11 165.1 0) (effects (font (size 1.016 1.016)) (hide yes)))
-(property "LCSC" "—" (at 118.11 165.1 0) (effects (font (size 1.016 1.016)) (hide yes)))
-(property "LCSC Part #" "—" (at 118.11 165.1 0) (effects (font (size 1.016 1.016)) (hide yes)))
-(property "Assembly" "Pads" (at 118.11 165.1 0) (effects (font (size 1.016 1.016)) (hide yes)))
-(property "Package" "5 SMD pads" (at 118.11 165.1 0) (effects (font (size 1.016 1.016)) (hide yes)))
-(property "Rating/Tolerance" "—" (at 118.11 165.1 0) (effects (font (size 1.016 1.016)) (hide yes)))
-(property "Source" "PCB copper" (at 118.11 165.1 0) (effects (font (size 1.016 1.016)) (hide yes)))
-(property "Workbook Value" "—" (at 118.11 165.1 0) (effects (font (size 1.016 1.016)) (hide yes)))
+(property "Value" "X6511WVS-05H-C60D48R1" (at 118.11 172.72 0) (effects (font (size 0.889 0.889))))
+(property "Footprint" "DAC_HPA:PinHeader_1x05_P2.54mm_SMD_XKB_X6511WVS-05H-C60D48R1" (at 118.11 165.1 0) (effects (font (size 1.016 1.016)) (hide yes)))
+(property "Datasheet" "https://www.lcsc.com/datasheet/C2883802.pdf" (at 118.11 165.1 0) (effects (font (size 1.016 1.016)) (hide yes)))
+(property "MPN" "XKB X6511WVS-05H-C60D48R1" (at 118.11 165.1 0) (effects (font (size 1.016 1.016)) (hide yes)))
+(property "LCSC" "C2883802" (at 118.11 165.1 0) (effects (font (size 1.016 1.016)) (hide yes)))
+(property "LCSC Part #" "C2883802" (at 118.11 165.1 0) (effects (font (size 1.016 1.016)) (hide yes)))
+(property "Assembly" "Yes" (at 118.11 165.1 0) (effects (font (size 1.016 1.016)) (hide yes)))
+(property "Package" "SMD 1x5 P2.54 mm vertical, staggered legs" (at 118.11 165.1 0) (effects (font (size 1.016 1.016)) (hide yes)))
+(property "Rating/Tolerance" "3 A, 250 V; 2.5 mm body, 6.0 mm mating pin" (at 118.11 165.1 0) (effects (font (size 1.016 1.016)) (hide yes)))
+(property "Source" "JLCPCB C2883802; order availability recheck" (at 118.11 165.1 0) (effects (font (size 1.016 1.016)) (hide yes)))
+(property "Workbook Value" "X6511WVS-05H-C60D48R1" (at 118.11 165.1 0) (effects (font (size 1.016 1.016)) (hide yes)))
 (property "Footprint status" "VERIFY G-3" (at 118.11 165.1 0) (effects (font (size 1.016 1.016)) (hide yes)))
 (pin "1")

Commit message: feat: CPLD pin reassignment ECO F06 for routability
AGRV2K U202 I/O moved to face their destinations: LINK_FRAME 11->26 and
LINK_MOSI 10->27 (north, toward U208), LINK_MISO 12->5 and CPLD_IRQ 14->7
(west, toward U201). Captured as a schematic overlay with an approved delta;
the board replay gains renamed_pads. CPLD RTL constraints must follow.
VALIDATE_OK, schematic checks pass, 0 DRC.

Co-Authored-By: Claude Opus 5.5 <noreply@anthropic.com>
Connections:
- net CPLD_IRQ: now also U202.7 (IO/PIN_7); no longer U202.14 (IO/PIN_14)
- net LINK_FRAME: now also U202.26 (IO/PIN_26); no longer U202.11 (IO/PIN_11)
- net LINK_MISO: now also U202.5 (IO/PIN_5); no longer U202.12 (IO/PIN_12)
- net LINK_MOSI: now also U202.27 (IO/PIN_27); no longer U202.10 (IO/PIN_10)
Changed lines of the file:
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@@
 (wire (pts (xy 120.65 71.12) (xy 118.11 71.12)) (stroke (width 0) (type solid)))
 (global_label "CPLD_NRST" (shape bidirectional) (at 118.11 71.12 180) (effects (font (size 0.762 0.762)) (justify right bottom)))
-(no_connect (at 120.65 73.66))
+(wire (pts (xy 120.65 73.66) (xy 118.11 73.66)) (stroke (width 0) (type solid)))
+(global_label "LINK_MISO" (shape bidirectional) (at 118.11 73.66 180) (effects (font (size 0.762 0.762)) (justify right bottom)))
 (wire (pts (xy 120.65 76.2) (xy 118.11 76.2)) (stroke (width 0) (type solid)))
 (global_label "N2_V33_CPLD" (shape bidirectional) (at 118.11 76.2 180) (effects (font (size 0.762 0.762)) (justify right bottom)))
-(no_connect (at 120.65 78.74))
+(wire (pts (xy 120.65 78.74) (xy 118.11 78.74)) (stroke (width 0) (type solid)))
+(global_label "CPLD_IRQ" (shape bidirectional) (at 118.11 78.74 180) (effects (font (size 0.762 0.762)) (justify right bottom)))
 (no_connect (at 120.65 81.28))
 (wire (pts (xy 120.65 83.82) (xy 118.11 83.82)) (stroke (width 0) (type solid)))
 (global_label "LINK_SCK" (shape bidirectional) (at 118.11 83.82 180) (effects (font (size 0.762 0.762)) (justify right bottom)))
-(wire (pts (xy 120.65 86.36) (xy 118.11 86.36)) (stroke (width 0) (type solid)))
-(global_label "LINK_MOSI" (shape bidirectional) (at 118.11 86.36 180) (effects (font (size 0.762 0.762)) (justify right bottom)))
-(wire (pts (xy 120.65 88.9) (xy 118.11 88.9)) (stroke (width 0) (type solid)))
-(global_label "LINK_FRAME" (shape bidirectional) (at 118.11 88.9 180) (effects (font (size 0.762 0.762)) (justify right bottom)))
-(wire (pts (xy 120.65 91.44) (xy 118.11 91.44)) (stroke (width 0) (type solid)))
-(global_label "LINK_MISO" (shape bidirectional) (at 118.11 91.44 180) (effects (font (size 0.762 0.762)) (justify right bottom)))
+(no_connect (at 120.65 86.36))
+(no_connect (at 120.65 88.9))
+(no_connect (at 120.65 91.44))
 (wire (pts (xy 120.65 93.98) (xy 118.11 93.98)) (stroke (width 0) (type solid)))
 (global_label "LRCLK_FB" (shape bidirectional) (at 118.11 93.98 180) (effects (font (size 0.762 0.762)) (justify right bottom)))
-(wire (pts (xy 120.65 96.52) (xy 118.11 96.52)) (stroke (width 0) (type solid)))
-(global_label "CPLD_IRQ" (shape bidirectional) (at 118.11 96.52 180) (effects (font (size 0.762 0.762)) (justify right bottom)))
+(no_connect (at 120.65 96.52))
 (no_connect (at 120.65 99.06))
 (wire (pts (xy 120.65 101.6) (xy 118.11 101.6)) (stroke (width 0) (type solid)))
@@
 (wire (pts (xy 171.45 81.28) (xy 173.99 81.28)) (stroke (width 0) (type solid)))
 (global_label "CPLD_JTCK" (shape bidirectional) (at 173.99 81.28 0) (effects (font (size 0.762 0.762)) (justify left bottom)))
-(no_connect (at 171.45 83.82))
-(no_connect (at 171.45 86.36))
+(wire (pts (xy 171.45 83.82) (xy 173.99 83.82)) (stroke (width 0) (type solid)))
+(global_label "LINK_FRAME" (shape bidirectional) (at 173.99 83.82 0) (effects (font (size 0.762 0.762)) (justify left bottom)))
+(wire (pts (xy 171.45 86.36) (xy 173.99 86.36)) (stroke (width 0) (type solid)))
+(global_label "LINK_MOSI" (shape bidirectional) (at 173.99 86.36 0) (effects (font (size 0.762 0.762)) (justify left bottom)))
 (no_connect (at 171.45 88.9))
 (no_connect (at 171.45 91.44))

Commit message: feat: CPLD pin ECO F06 v2 and FAM_CLK corridor; 64 ratsnest links
F06 v2 moves every reassignable AGRV2K signal off the west row, which FAM_CLK
and its L2-protection via keep-out seal: LINK_FRAME/MOSI/MISO, CPLD_IRQ and
OSC48_EN to the north row, OSC44_EN to pin 8. R215 stands level with pin 1 so
FAM_CLK is a straight 1.5 mm run, opening a via site beside CPLD_NRST.
Freerouting rounds re-routed plain control nets; VREF keeps its hand route.
VALIDATE_OK, schematic checks pass, 0 DRC. CPLD RTL constraints must follow.

Co-Authored-By: Claude Opus 5.5 <noreply@anthropic.com>
Connections:
- net CPLD_IRQ: now also U202.29 (IO/PIN_29); no longer U202.7 (IO/PIN_7)
- net LINK_MISO: now also U202.28 (IO/PIN_28); no longer U202.5 (IO/PIN_5)
- net OSC44_EN: now also U202.8 (IO/PIN_8); no longer U202.3 (IO/PIN_3)
- net OSC48_EN: now also U202.31 (IO/PIN_31); no longer U202.2 (IO/PIN_2)
Changed lines of the file:
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@@
 (wire (pts (xy 120.65 63.5) (xy 118.11 63.5)) (stroke (width 0) (type solid)))
 (global_label "FAM_CLK" (shape bidirectional) (at 118.11 63.5 180) (effects (font (size 0.762 0.762)) (justify right bottom)))
-(wire (pts (xy 120.65 66.04) (xy 118.11 66.04)) (stroke (width 0) (type solid)))
-(global_label "OSC48_EN" (shape bidirectional) (at 118.11 66.04 180) (effects (font (size 0.762 0.762)) (justify right bottom)))
-(wire (pts (xy 120.65 68.58) (xy 118.11 68.58)) (stroke (width 0) (type solid)))
-(global_label "OSC44_EN" (shape bidirectional) (at 118.11 68.58 180) (effects (font (size 0.762 0.762)) (justify right bottom)))
+(no_connect (at 120.65 66.04))
+(no_connect (at 120.65 68.58))
 (wire (pts (xy 120.65 71.12) (xy 118.11 71.12)) (stroke (width 0) (type solid)))
 (global_label "CPLD_NRST" (shape bidirectional) (at 118.11 71.12 180) (effects (font (size 0.762 0.762)) (justify right bottom)))
-(wire (pts (xy 120.65 73.66) (xy 118.11 73.66)) (stroke (width 0) (type solid)))
-(global_label "LINK_MISO" (shape bidirectional) (at 118.11 73.66 180) (effects (font (size 0.762 0.762)) (justify right bottom)))
+(no_connect (at 120.65 73.66))
 (wire (pts (xy 120.65 76.2) (xy 118.11 76.2)) (stroke (width 0) (type solid)))
 (global_label "N2_V33_CPLD" (shape bidirectional) (at 118.11 76.2 180) (effects (font (size 0.762 0.762)) (justify right bottom)))
-(wire (pts (xy 120.65 78.74) (xy 118.11 78.74)) (stroke (width 0) (type solid)))
-(global_label "CPLD_IRQ" (shape bidirectional) (at 118.11 78.74 180) (effects (font (size 0.762 0.762)) (justify right bottom)))
-(no_connect (at 120.65 81.28))
+(no_connect (at 120.65 78.74))
+(wire (pts (xy 120.65 81.28) (xy 118.11 81.28)) (stroke (width 0) (type solid)))
+(global_label "OSC44_EN" (shape bidirectional) (at 118.11 81.28 180) (effects (font (size 0.762 0.762)) (justify right bottom)))
 (wire (pts (xy 120.65 83.82) (xy 118.11 83.82)) (stroke (width 0) (type solid)))
 (global_label "LINK_SCK" (shape bidirectional) (at 118.11 83.82 180) (effects (font (size 0.762 0.762)) (justify right bottom)))
@@
 (wire (pts (xy 171.45 86.36) (xy 173.99 86.36)) (stroke (width 0) (type solid)))
 (global_label "LINK_MOSI" (shape bidirectional) (at 173.99 86.36 0) (effects (font (size 0.762 0.762)) (justify left bottom)))
-(no_connect (at 171.45 88.9))
-(no_connect (at 171.45 91.44))
+(wire (pts (xy 171.45 88.9) (xy 173.99 88.9)) (stroke (width 0) (type solid)))
+(global_label "LINK_MISO" (shape bidirectional) (at 173.99 88.9 0) (effects (font (size 0.762 0.762)) (justify left bottom)))
+(wire (pts (xy 171.45 91.44) (xy 173.99 91.44)) (stroke (width 0) (type solid)))
+(global_label "CPLD_IRQ" (shape bidirectional) (at 173.99 91.44 0) (effects (font (size 0.762 0.762)) (justify left bottom)))
 (wire (pts (xy 171.45 93.98) (xy 173.99 93.98)) (stroke (width 0) (type solid)))
 (global_label "GND" (shape bidirectional) (at 173.99 93.98 0) (effects (font (size 0.762 0.762)) (justify left bottom)))
-(no_connect (at 171.45 96.52))
+(wire (pts (xy 171.45 96.52) (xy 173.99 96.52)) (stroke (width 0) (type solid)))
+(global_label "OSC48_EN" (shape bidirectional) (at 173.99 96.52 0) (effects (font (size 0.762 0.762)) (justify left bottom)))
 (wire (pts (xy 171.45 99.06) (xy 173.99 99.06)) (stroke (width 0) (type solid)))
 (global_label "N2_V33_CPLD" (shape bidirectional) (at 173.99 99.06 0) (effects (font (size 0.762 0.762)) (justify left bottom)))

Commit message: feat: ECO F07, CPLD-driven I2S capture copies; 28 ratsnest links
Owner decision: the 330 ohm bit-perfect capture taps R228-R230 could not branch
from the side-by-side, F.Cu-only N2_*_SRC lines at the CPLD end. U202 now drives
dedicated copies on spare pins 22/15/23 (N2_CPY_CK/WS/SD) into R228/R229/R230 as
source series resistors; pad 2 still feeds N2_CAP_* to PB13/PB12/PB15. The DAC
lines carry no capture stubs. The RTL must duplicate the three I2S output
registers onto the copy pins.

- Schematic: asserted overlay in generate_schematic.py, approved delta in
  verify_schematic.py, net counts 250 -> 253 in the verifiers.
- Board: block 76 with added_nets and renamed_pads (replay support added).
- TP717 moves onto the SDATA run (zero stub). R224 stays at the MCU per the
  design notes, sharing the pocket with R216; X203's supply via moves to its pad.
- R218.2 is re-tied to C218.2 after a router path split its pour.

28 links, 0 DRC, VALIDATE_OK, schematic checks PASS, high-Z deviation pairs 28.

Co-Authored-By: Claude Opus 5.5 <noreply@anthropic.com>
Connections:
- net N2_BCLK_SRC: no longer R228.1
- net N2_LRCLK_SRC: no longer R229.1
- net N2_SDATA_SRC: no longer R230.1
- net N2_CPY_WS: now reaches U202.15 (IO/PIN_15)
- net N2_CPY_WS: now also R229.1
- net N2_CPY_CK: now reaches U202.22 (IO/PIN_22)
- net N2_CPY_CK: now also R228.1
- net N2_CPY_SD: now reaches U202.23 (IO/PIN_23)
- net N2_CPY_SD: now also R230.1
- no-connect marks 11 -> 8
Changed lines of the file:
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@@
 )
 (wire (pts (xy 91.44 308.61) (xy 88.9 308.61)) (stroke (width 0) (type solid)))
-(global_label "N2_BCLK_SRC" (shape bidirectional) (at 88.9 308.61 180) (effects (font (size 0.762 0.762)) (justify right bottom)))
+(global_label "N2_CPY_CK" (shape bidirectional) (at 88.9 308.61 180) (effects (font (size 0.762 0.762)) (justify right bottom)))
 (wire (pts (xy 101.6 308.61) (xy 104.14 308.61)) (stroke (width 0) (type solid)))
 (global_label "N2_CAP_CK" (shape bidirectional) (at 104.14 308.61 0) (effects (font (size 0.762 0.762)) (justify left bottom)))
@@
 )
 (wire (pts (xy 137.16 308.61) (xy 134.62 308.61)) (stroke (width 0) (type solid)))
-(global_label "N2_LRCLK_SRC" (shape bidirectional) (at 134.62 308.61 180) (effects (font (size 0.762 0.762)) (justify right bottom)))
+(global_label "N2_CPY_WS" (shape bidirectional) (at 134.62 308.61 180) (effects (font (size 0.762 0.762)) (justify right bottom)))
 (wire (pts (xy 147.32 308.61) (xy 149.86 308.61)) (stroke (width 0) (type solid)))
 (global_label "N2_CAP_WS" (shape bidirectional) (at 149.86 308.61 0) (effects (font (size 0.762 0.762)) (justify left bottom)))
@@
 )
 (wire (pts (xy 182.88 308.61) (xy 180.34 308.61)) (stroke (width 0) (type solid)))
-(global_label "N2_SDATA_SRC" (shape bidirectional) (at 180.34 308.61 180) (effects (font (size 0.762 0.762)) (justify right bottom)))
+(global_label "N2_CPY_SD" (shape bidirectional) (at 180.34 308.61 180) (effects (font (size 0.762 0.762)) (justify right bottom)))
 (wire (pts (xy 193.04 308.61) (xy 195.58 308.61)) (stroke (width 0) (type solid)))
 (global_label "N2_CAP_SD" (shape bidirectional) (at 195.58 308.61 0) (effects (font (size 0.762 0.762)) (justify left bottom)))
@@
 (global_label "LRCLK_FB" (shape bidirectional) (at 118.11 93.98 180) (effects (font (size 0.762 0.762)) (justify right bottom)))
 (no_connect (at 120.65 96.52))
-(no_connect (at 120.65 99.06))
+(wire (pts (xy 120.65 99.06) (xy 118.11 99.06)) (stroke (width 0) (type solid)))
+(global_label "N2_CPY_WS" (shape bidirectional) (at 118.11 99.06 180) (effects (font (size 0.762 0.762)) (justify right bottom)))
 (wire (pts (xy 120.65 101.6) (xy 118.11 101.6)) (stroke (width 0) (type solid)))
 (global_label "N2_V33_CPLD" (shape bidirectional) (at 118.11 101.6 180) (effects (font (size 0.762 0.762)) (justify right bottom)))
@@
 (wire (pts (xy 171.45 71.12) (xy 173.99 71.12)) (stroke (width 0) (type solid)))
 (global_label "MCLK_EN" (shape bidirectional) (at 173.99 71.12 0) (effects (font (size 0.762 0.762)) (justify left bottom)))
-(no_connect (at 171.45 73.66))
-(no_connect (at 171.45 76.2))
+(wire (pts (xy 171.45 73.66) (xy 173.99 73.66)) (stroke (width 0) (type solid)))
+(global_label "N2_CPY_CK" (shape bidirectional) (at 173.99 73.66 0) (effects (font (size 0.762 0.762)) (justify left bottom)))
+(wire (pts (xy 171.45 76.2) (xy 173.99 76.2)) (stroke (width 0) (type solid)))
+(global_label "N2_CPY_SD" (shape bidirectional) (at 173.99 76.2 0) (effects (font (size 0.762 0.762)) (justify left bottom)))
 (wire (pts (xy 171.45 78.74) (xy 173.99 78.74)) (stroke (width 0) (type solid)))
 (global_label "CPLD_JTMS" (shape bidirectional) (at 173.99 78.74 0) (effects (font (size 0.762 0.762)) (justify left bottom)))

Commit message: fix: ECO F07 revision - WS capture taps LRCLK_FB; drop the third CPLD copy pin
R229.1 joins LRCLK_FB (U202 pin 13, already an LRCLK copy from its own
output register, routed to MCU PD2). Pin 15 returns to NC and N2_CPY_WS
is deleted, so the CPLD RTL needs only pins 22 (BCLK copy) and 23 (SDATA
copy). Schematic regenerated; verify_schematic / verify_design_notes /
validate_integrated_audio_study pass (252 named nets). Board: 0 DRC, 9 links.

Co-Authored-By: Claude Opus 5.5 <noreply@anthropic.com>
Connections:
- net LRCLK_FB: now also R229.1
- net N2_CPY_WS: no longer names the net of U202.15 (IO/PIN_15)
- net N2_CPY_WS: no longer R229.1
- no-connect marks 8 -> 9
Changed lines of the file:
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@@
 )
 (wire (pts (xy 137.16 308.61) (xy 134.62 308.61)) (stroke (width 0) (type solid)))
-(global_label "N2_CPY_WS" (shape bidirectional) (at 134.62 308.61 180) (effects (font (size 0.762 0.762)) (justify right bottom)))
+(global_label "LRCLK_FB" (shape bidirectional) (at 134.62 308.61 180) (effects (font (size 0.762 0.762)) (justify right bottom)))
 (wire (pts (xy 147.32 308.61) (xy 149.86 308.61)) (stroke (width 0) (type solid)))
 (global_label "N2_CAP_WS" (shape bidirectional) (at 149.86 308.61 0) (effects (font (size 0.762 0.762)) (justify left bottom)))
@@
 (global_label "LRCLK_FB" (shape bidirectional) (at 118.11 93.98 180) (effects (font (size 0.762 0.762)) (justify right bottom)))
 (no_connect (at 120.65 96.52))
-(wire (pts (xy 120.65 99.06) (xy 118.11 99.06)) (stroke (width 0) (type solid)))
-(global_label "N2_CPY_WS" (shape bidirectional) (at 118.11 99.06 180) (effects (font (size 0.762 0.762)) (justify right bottom)))
+(no_connect (at 120.65 99.06))
 (wire (pts (xy 120.65 101.6) (xy 118.11 101.6)) (stroke (width 0) (type solid)))
 (global_label "N2_V33_CPLD" (shape bidirectional) (at 118.11 101.6 180) (effects (font (size 0.762 0.762)) (justify right bottom)))
