File: hardware/02_usb_bridge.kicad_sch (KiCad schematic)
At the start: 73 parts, among them J201 X6511WVS-08H-C60D48R1, J202 X6511WVS-05H-C60D48R1, Q207 AO3400A, U201 CH32V307RCT6, U202 AGRV2KQ32, U205 74LVC1G157, U206 74LVC1G11, U208 74LVC3G34, X201 80.000 MHz, X202 49.152 MHz, X203 45.1584 MHz, Y201 8 MHz

Commit message: feat: route all held nets; ECO F08 CPLD pin rotation; DC_SENSE_LP off the U201 pin row; 9 plain links
- R690 (N6_TRIP pull-up) and R693/R694 (HREF divider) moved beside U606;
  REF13 / V13_CMP / N6_H links re-routed (layout only).
- DC_SENSE_LP leaves F.Cu along U201's east pin row (it blocked every via
  site for pins 17-32); runs on L4, length unchanged.
- ECO F08: U202 IO pins 21/22/23 = N2_CPY_CK / N2_CPY_SD / MCLK_EN (RTL pin
  constraint change; schematic overlay + approved delta).
- MCU/CPLD group (CPLD_NRST, LRCLK_FB + WS tap, F07 copies, LINK bus,
  N6_ARM_MCU, N2_DCS_RN_PIN) routed jointly; Freerouting rounds 19-20 re-routed
  the plain nets around it.

0 DRC, 9 ratsnest links (all plain digital control nets), VALIDATE_OK,
schematic checks pass, high-Z deviation pairs 30.

Co-Authored-By: Claude Opus 5.5 <noreply@anthropic.com>
Connections:
- net MCLK_EN: now also U202.23 (IO/PIN_23); no longer U202.21 (IO/PIN_21)
- net N2_CPY_CK: now also U202.21 (IO/PIN_21); no longer U202.22 (IO/PIN_22)
- net N2_CPY_SD: now also U202.22 (IO/PIN_22); no longer U202.23 (IO/PIN_23)
Changed lines of the file:
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@@
 (global_label "N2_SDATA_SRC" (shape bidirectional) (at 173.99 68.58 0) (effects (font (size 0.762 0.762)) (justify left bottom)))
 (wire (pts (xy 171.45 71.12) (xy 173.99 71.12)) (stroke (width 0) (type solid)))
-(global_label "MCLK_EN" (shape bidirectional) (at 173.99 71.12 0) (effects (font (size 0.762 0.762)) (justify left bottom)))
+(global_label "N2_CPY_CK" (shape bidirectional) (at 173.99 71.12 0) (effects (font (size 0.762 0.762)) (justify left bottom)))
 (wire (pts (xy 171.45 73.66) (xy 173.99 73.66)) (stroke (width 0) (type solid)))
-(global_label "N2_CPY_CK" (shape bidirectional) (at 173.99 73.66 0) (effects (font (size 0.762 0.762)) (justify left bottom)))
+(global_label "N2_CPY_SD" (shape bidirectional) (at 173.99 73.66 0) (effects (font (size 0.762 0.762)) (justify left bottom)))
 (wire (pts (xy 171.45 76.2) (xy 173.99 76.2)) (stroke (width 0) (type solid)))
-(global_label "N2_CPY_SD" (shape bidirectional) (at 173.99 76.2 0) (effects (font (size 0.762 0.762)) (justify left bottom)))
+(global_label "MCLK_EN" (shape bidirectional) (at 173.99 76.2 0) (effects (font (size 0.762 0.762)) (justify left bottom)))
 (wire (pts (xy 171.45 78.74) (xy 173.99 78.74)) (stroke (width 0) (type solid)))
 (global_label "CPLD_JTMS" (shape bidirectional) (at 173.99 78.74 0) (effects (font (size 0.762 0.762)) (justify left bottom)))
