File: hardware/01_usb_input.kicad_sch (KiCad schematic)
At the start: 18 parts, among them J101 GCT USB4105-GF-A, U101 ST USBLC6-2SC6, U102 TI TPS25200DRVR, U103 TI TPD2E2U06DRLR

Commit message: fix: keep the frozen study boards' J101 library footprint; corrected lands as J101_..._NPTH030
The previous commit edited the shared J101 footprint in place, so every frozen study board that embeds
the original reported lib_footprint_mismatch in KiCad DRC (CI: macro, output macro, functional ECO,
discharge fit, manual review). The original footprint is restored unchanged; the 0.98 mm-land version
is J101_USB4105-GF-A_12lands_4stakes_NPTH030, used by the schematic, BOM, G-3 overlay and the
integrated board (J101 joins the post-freeze ECO refs for the frozen boards' netlist check).
Frozen boards: KiCad DRC 0 again. Integrated board: DRC 0, VALIDATE_OK.

Also corrects the result count in the previous commit message and response document: the
sign-off suite ends at 0 FAIL / 10 WARN / 9 PASS (not 11 / 8).

Co-Authored-By: Claude Opus 5.5 <noreply@anthropic.com>
Parts:
- J101: footprint DAC_HPA:J101_USB4105-GF-A_12lands_4stakes -> DAC_HPA:J101_USB4105-GF-A_12lands_4stakes_NPTH030
Changed lines of the file:
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@@
 (property "Reference" "J101" (at 60.96 58.42 0) (effects (font (size 0.889 0.889))))
 (property "Value" "GCT USB4105-GF-A" (at 60.96 86.36 0) (effects (font (size 0.889 0.889))))
-(property "Footprint" "DAC_HPA:J101_USB4105-GF-A_12lands_4stakes" (at 60.96 72.39 0) (effects (font (size 1.016 1.016)) (hide yes)))
+(property "Footprint" "DAC_HPA:J101_USB4105-GF-A_12lands_4stakes_NPTH030" (at 60.96 72.39 0) (effects (font (size 1.016 1.016)) (hide yes)))
 (property "Datasheet" "https://gct.co/connector/usb4105 (drawing text: https://www.mouser.com/datasheet/2/837/USB4105-1948910.pdf)" (at 60.96 72.39 0) (effects (font (size 1.016 1.016)) (hide yes)))
 (property "MPN" "GCT USB4105-GF-A" (at 60.96 72.39 0) (effects (font (size 1.016 1.016)) (hide yes)))
